Commit message: Introduced differential control. Issues with turns

File: carmen_description/robot/carmen.gazebo.xacro (robot description, xacro)
@@ -14,186 +14,59 @@
         <material>Gazebo/White</material>
     </gazebo>
-    <gazebo reference="head_link">
-        <material>Gazebo/White</material>
-    </gazebo>
-    <gazebo reference="neck_link">
-        <material>Gazebo/White</material>
-    </gazebo>
-    <gazebo reference="camera_stick_link">
-        <material>Gazebo/Yellow</material>
-    </gazebo>
-    <gazebo reference="imu_link">
-        <material>Gazebo/Green</material>
-    </gazebo>
-    <gazebo reference="front_left_wheel_link">
-        <mu1>0.0</mu1>
-        <mu2>0.0</mu2>
-        <material>Gazebo/Blue</material>
-    </gazebo>
-    <gazebo reference="front_right_wheel_link">
-        <mu1>0.0</mu1>
-        <mu2>0.0</mu2>
-        <material>Gazebo/Blue</material>
-    </gazebo>
-    <gazebo reference="rear_left_wheel_link">
-        <mu1>0.0</mu1>
-        <mu2>0.0</mu2>
-        <material>Gazebo/Blue</material>
-    </gazebo>
-    <gazebo reference="rear_right_wheel_link">
-        <mu1>0.0</mu1>
-        <mu2>0.0</mu2>
-        <material>Gazebo/Blue</material>
-    </gazebo>
-    <gazebo reference="front_right_motor_holder">
+    <gazebo reference="front_left_wheel">
         <mu1 value="1.0"/>
         <mu2 value="1.0"/>
         <kp value="10000000.0"/>
         <kd value="1.0"/>
-        <material>Gazebo/Red</material>
+        <material>Gazebo/Black</material>
     </gazebo>
-    <gazebo reference="front_left_motor_holder">
+    <gazebo reference="front_right_wheel">
         <mu1 value="1.0"/>
         <mu2 value="1.0"/>
         <kp value="10000000.0"/>
         <kd value="1.0"/>
-        <material>Gazebo/Red</material>
+        <material>Gazebo/Black</material>
     </gazebo>
-    <gazebo reference="rear_left_motor_holder">
+    <gazebo reference="rear_left_wheel">
         <mu1 value="1.0"/>
         <mu2 value="1.0"/>
         <kp value="10000000.0"/>
         <kd value="1.0"/>
-        <material>Gazebo/Red</material>
+        <material>Gazebo/Black</material>
     </gazebo>
-    <gazebo reference="rear_right_motor_holder">
+    <gazebo reference="rear_right_wheel">
         <mu1 value="1.0"/>
         <mu2 value="1.0"/>
         <kp value="10000000.0"/>
         <kd value="1.0"/>
-        <material>Gazebo/Red</material>
+        <material>Gazebo/Black</material>
     </gazebo>
-    <gazebo reference="left_camera_link">
-        <material>Gazebo/Green</material>
-        <sensor type="multicamera" name="stereo_camera">
-            <update_rate>30.0</update_rate>
-            <camera name="left">
-                <horizontal_fov>1.3962634</horizontal_fov>
-                <image>
-                    <width>800</width>
-                    <height>800</height>
-                    <format>R8G8B8</format>
-                </image>
-                <clip>
-                    <near>0.02</near>
-                    <far>300</far>
-                </clip>
-                <noise>
-                    <type>gaussian</type>
-                    <mean>0.0</mean>
-                    <stddev>0.007</stddev>
-                </noise>
-            </camera>
-            <camera name="right">
-                <pose>0 -0.07 0 0 0 0</pose>
-                <horizontal_fov>1.3962634</horizontal_fov>
-                <image>
-                    <width>800</width>
-                    <height>800</height>
-                    <format>R8G8B8</format>
-                </image>
-                <clip>
-                    <near>0.02</near>
-                    <far>300</far>
-                </clip>
-                <noise>
-                    <type>gaussian</type>
-                    <mean>0.0</mean>
-                    <stddev>0.007</stddev>
-                </noise>
-            </camera>
-            <plugin name="stereo_camera_controller" filename="libgazebo_ros_multicamera.so">
-                <alwaysOn>true</alwaysOn>
-                <updateRate>0.0</updateRate>
-                <cameraName>stereocamera</cameraName>
-                <imageTopicName>image_raw</imageTopicName>
-                <cameraInfoTopicName>camera_info</cameraInfoTopicName>
-                <frameName>left_camera_link</frameName>
-                <rightFrameName>right_camera_link</rightFrameName>
-                <hackBaseline>0.07</hackBaseline>
-                <distortionK1>0.0</distortionK1>
-                <distortionK2>0.0</distortionK2>
-                <distortionK3>0.0</distortionK3>
-                <distortionT1>0.0</distortionT1>
-                <distortionT2>0.0</distortionT2>
-            </plugin>
-        </sensor>
+    <gazebo reference="front_right_bearing">
+        <mu1 value="1.0"/>
+        <mu2 value="1.0"/>
+        <kp value="10000000.0"/>
+        <kd value="1.0"/>
+        <material>Gazebo/Blue</material>
     </gazebo>
-    <gazebo reference="right_camera_link">
-        <material>Gazebo/Green</material>
+    <gazebo reference="front_left_bearing">
+        <mu1 value="1.0"/>
+        <mu2 value="1.0"/>
+        <kp value="10000000.0"/>
+        <kd value="1.0"/>
+        <material>Gazebo/Blue</material>
     </gazebo>
-    <!-- Hokuyo LIDAR for simulation -->
-    <gazebo reference="laser_link">
-        <material>Gazebo/Green</material>
-        <sensor type="ray" name="laser">
-            <pose>0 0 0 0 0 0</pose>
-            <visualize>false</visualize>
-            <update_rate>40</update_rate>
-            <ray>
-                <scan>
-                    <horizontal>
-                        <samples>1081</samples>
-                        <resolution>1</resolution>
-                        <min_angle>-1.570796</min_angle>
-                        <max_angle>1.570796</max_angle>
-                    </horizontal>
-                </scan>
-                <range>
-                    <min>0.60</min>
-                    <max>10.0</max>
-                    <resolution>0.01</resolution>
-                </range>
-                <noise>
-                    <type>gaussian</type>
-                    <mean>0.0</mean>
-                    <stddev>0.01</stddev>
-                </noise>
-            </ray>
-            <plugin name="gazebo_ros_hokuyo_controller" filename="libgazebo_ros_laser.so">
-                <topicName>laser/scan</topicName>
-                <frameName>laser_link</frameName>
-            </plugin>
-        </sensor>
+    <gazebo reference="rear_left_bearing">
+        <mu1 value="1.0"/>
+        <mu2 value="1.0"/>
+        <kp value="10000000.0"/>
+        <kd value="1.0"/>
+        <material>Gazebo/Blue</material>
     </gazebo>
-    <gazebo>
-        <plugin name="imu_controller" filename="libhector_gazebo_ros_imu.so">
-            <robotNamespace>/</robotNamespace>
-            <updateRate>50.0</updateRate>
-            <bodyName>base_footprint</bodyName>
-            <frameId>imu_link</frameId>
-            <topicName>imu/data</topicName>
-            <accelDrift>0.005 0.005 0.005</accelDrift>
-            <accelGaussianNoise>0.005 0.005 0.005</accelGaussianNoise>
-            <rateDrift>0.00005 0.00005 0.00005</rateDrift>
-            <rateGaussianNoise>0.00005 0.00005 0.00005</rateGaussianNoise>
-            <headingDrift>0.005</headingDrift>
-            <headingGaussianNoise>0.005</headingGaussianNoise>
-        </plugin>
-    </gazebo>
-    <gazebo>
-         <plugin name="ridgeback_ros_force_based_move" filename="libridgeback_ros_force_based_move.so">
-            <robotNamespace>/</robotNamespace>
-            <commandTopic>/mecanum_velocity_controller/cmd_vel</commandTopic>
-            <odometryTopic>odom</odometryTopic>
-            <odometryFrame>odom</odometryFrame>
-            <odometryRate>25.0</odometryRate>
-            <robotBaseFrame>base_footprint</robotBaseFrame>
-            <cmdVelTimeOut>0.25</cmdVelTimeOut>
-            <!-- Don't publish a transform: the controller does it. -->
-            <publishOdometryTf>0</publishOdometryTf>
-            <yaw_velocity_p_gain>100.0</yaw_velocity_p_gain>
-            <x_velocity_p_gain>100.0</x_velocity_p_gain>
-            <y_velocity_p_gain>100.0</y_velocity_p_gain>
-        </plugin>
+    <gazebo reference="rear_right_bearing">
+        <mu1 value="1.0"/>
+        <mu2 value="1.0"/>
+        <kp value="10000000.0"/>
+        <kd value="1.0"/>
+        <material>Gazebo/Blue</material>
     </gazebo>
 </robot>

File: carmen_description/robot/robot.urdf.xacro (robot description, xacro)
@@ -4,12 +4,12 @@
   <xacro:include filename="$(find carmen_description)/urdf/sensors/camera.urdf.xacro"/>
   <xacro:include filename="$(find carmen_description)/urdf/wheels.urdf.xacro"/>
-  <xacro:property name="base_width" value="0.2"/>
-  <xacro:property name="base_length" value="0.25"/>
-  <xacro:property name="base_height" value="0.1"/>
+  <xacro:property name="base_width" value="0.3"/>
+  <xacro:property name="base_length" value="0.2"/>
+  <xacro:property name="base_height" value="0.05"/>
   <xacro:property name="base_mass" value="0.4"/>
-  <xacro:property name="wheel_width" value="0.035"/>
-  <xacro:property name="wheel_radius" value="0.1"/>
-  <xacro:property name="wheel_mass" value="10"/>
-  <xacro:property name="bearing_radius" value="0.01"/>
+  <xacro:property name="wheel_width" value="0.02"/>
+  <xacro:property name="wheel_radius" value="0.035"/>
+  <xacro:property name="wheel_mass" value="1"/>
+  <xacro:property name="bearing_radius" value="0.005"/>
   <link name="base_footprint"/>
   <joint name="base_footprint_joint" type="fixed">
@@ -27,14 +27,14 @@
   </link>
   <xacro:wheel prefix="front_left" direction="1" bearing_radius="${bearing_radius}" radius="${wheel_radius}"
-               width="${wheel_width}" mass="${wheel_mass}" distance_between_wheels="${base_width}"
-               x="${base_width / 4}" z="0"/>
+               width="${wheel_width}" mass="${wheel_mass}" distance_between_wheels="${base_length}"
+               x="${base_width / 4}" z="${bearing_radius - base_height / 2}"/>
   <xacro:wheel prefix="front_right" direction="-1" bearing_radius="${bearing_radius}" radius="${wheel_radius}"
-               width="${wheel_width}" mass="${wheel_mass}" distance_between_wheels="${base_width}"
-               x="${base_width / 4}" z="0"/>
+               width="${wheel_width}" mass="${wheel_mass}" distance_between_wheels="${base_length}"
+               x="${base_width / 4}" z="${bearing_radius - base_height / 2}"/>
   <xacro:wheel prefix="rear_left" direction="1" bearing_radius="${bearing_radius}" radius="${wheel_radius}"
-               width="${wheel_width}" mass="${wheel_mass}" distance_between_wheels="${base_width}"
-               x="${-base_width / 4}" z="0"/>
+               width="${wheel_width}" mass="${wheel_mass}" distance_between_wheels="${base_length}"
+               x="${-base_width / 4}" z="${bearing_radius - base_height / 2}"/>
   <xacro:wheel prefix="rear_right" direction="-1" bearing_radius="${bearing_radius}" radius="${wheel_radius}"
-               width="${wheel_width}" mass="${wheel_mass}" distance_between_wheels="${base_width}"
-               x="${-base_width / 4}" z="0"/>
+               width="${wheel_width}" mass="${wheel_mass}" distance_between_wheels="${base_length}"
+               x="${-base_width / 4}" z="${bearing_radius - base_height / 2}"/>
 </robot>

File: carmen_description/urdf/wheels.urdf.xacro (robot description, xacro)
@@ -2,5 +2,5 @@
   <xacro:macro name="wheel"
          params="prefix direction bearing_radius radius width mass distance_between_wheels x z">
-    <link name="${prefix}_bearing_link">>
+    <link name="${prefix}_bearing">
       <visual>
         <xacro:cylinder_geometry radius="${bearing_radius}" height="${2 * wheel_width}"/>
@@ -14,31 +14,30 @@
           xyz="${x} ${direction * (distance_between_wheels/2 + wheel_width)} ${z}"/>
       <parent link="base_link"/>
-      <child link="${prefix}_bearing_link"/>
+      <child link="${prefix}_bearing"/>
     </joint>
-    <link name="${prefix}_wheel_link">
+    <link name="${prefix}_wheel">
       <visual>
-        <origin rpy="${pi / 2} 0 0 " xyz="0 0 0"/>
+        <origin rpy="0 0 0 " xyz="0 0 0"/>
           <xacro:cylinder_geometry radius="${radius}" height="${width}"/>
-          <xacro:blue_material/>
-        <xacro:red_material/>
+          <xacro:black_material/>
       </visual>
       <xacro:cylinder_collision radius="${radius}" height="${width}"/>
       <xacro:cylinder_inertia mass="${mass}" radius="${radius}" height="${width}"/>
     </link>
-    <joint name="${prefix}_wheel_bearing_joint" type="continuous">
+    <joint name="${prefix}_wheel_joint" type="continuous">
       <origin rpy="0 0 0" xyz="0 0 ${direction * wheel_width/2}"/>
-      <parent link="${prefix}_bearing_link"/>
-      <child link="${prefix}_wheel_link"/>
+      <parent link="${prefix}_bearing"/>
+      <child link="${prefix}_wheel"/>
       <axis xyz="0 0 1"/>
     </joint>
     <transmission name="${prefix}_wheel_transmission">
       <type>transmission_interface/SimpleTransmission</type>
-      <joint name="${prefix}_wheel_bearing_joint">
+      <joint name="${prefix}_wheel_joint">
         <hardwareInterface>hardware_interface/VelocityJointInterface</hardwareInterface>
       </joint>
       <actuator name="${prefix}_wheel_motor">
         <hardwareInterface>hardware_interface/VelocityJointInterface</hardwareInterface>
-        <mechanicalReduction>500</mechanicalReduction>
-        <motorTorqueConstant>0.5</motorTorqueConstant>
+        <mechanicalReduction>1</mechanicalReduction>
+        <motorTorqueConstant>1</motorTorqueConstant>
       </actuator>
     </transmission>

Commit message: Added visualization of sonar, camera and IMU.

File: carmen_description/robot/carmen.gazebo.xacro (robot description, xacro)
@@ -12,5 +12,5 @@
     </gazebo>
     <gazebo reference="base_link">
-        <material>Gazebo/White</material>
+        <material>Gazebo/Yellow</material>
     </gazebo>
     <gazebo reference="front_left_wheel">
@@ -74,3 +74,18 @@
         <material>Gazebo/Blue</material>
     </gazebo>
+    <gazebo reference="left_sonar_link">
+        <material>Gazebo/White</material>
+    </gazebo>
+    <gazebo reference="right_sonar_link">
+        <material>Gazebo/White</material>
+    </gazebo>
+    <gazebo reference="left_camera_link">
+        <material>Gazebo/Green</material>
+    </gazebo>
+    <gazebo reference="right_camera_link">
+        <material>Gazebo/Green</material>
+    </gazebo>
+    <gazebo reference="imu_link">
+        <material>Gazebo/Black</material>
+    </gazebo>
 </robot>

File: carmen_description/robot/robot.urdf.xacro (robot description, xacro)
@@ -12,4 +12,6 @@
   <xacro:property name="wheel_radius" value="0.035"/>
   <xacro:property name="wheel_mass" value="1"/>
+  <xacro:property name="imu_size" value="0.01"/>
+  <xacro:property name="imu_mass" value="0.01"/>
   <xacro:property name="bearing_radius" value="0.005"/>
   <link name="base_footprint"/>
@@ -27,8 +29,25 @@
     <xacro:box_inertia width="${base_width}" length="${base_length}" height="${base_height}" mass="${base_mass}"/>
   </link>
+  <link name="imu_link">
+    <visual>
+      <xacro:cube_geometry size="${imu_size}"/>
+      <xacro:black_material/>
+    </visual>
+    <xacro:cube_collision size="${imu_size}"/>
+    <xacro:cube_inertia mass="${imu_mass}" size="${imu_size}"/>
+  </link>
+  <joint name="imu_joint" type="fixed">
+      <origin xyz="-0.025 0 ${(base_height + imu_size) / 2}" rpy="0 0 0"/>
+      <parent link="base_link"/>
+      <child link="imu_link"/>
+  </joint>
   <xacro:simple_camera prefix="left" parent_link_name="base_link" parent_height="${base_height}"
-                       parent_length="${base_length / 2}" side="1"/>
+                       parent_length="${base_length / 2}" side="1" x="${base_width / 2}"/>
   <xacro:simple_camera prefix="right" parent_link_name="base_link" parent_height="${base_height}"
-                       parent_length="${base_length / 2}" side="-1"/>
+                       parent_length="${base_length / 2}" side="-1" x="${base_width / 2}"/>
+  <xacro:simple_sonar prefix="left" parent_link_name="base_link" x="${base_width / 2}" y="${base_length / 2}"
+                      z="${base_height / 2}"/>
+  <xacro:simple_sonar prefix="right" parent_link_name="base_link" x="${base_width / 2}" y="${-base_length / 2}"
+                      y_side="-1" z="${base_height / 2}"/>
   <xacro:wheel prefix="front_left" direction="1" bearing_radius="${bearing_radius}" radius="${wheel_radius}"
                width="${wheel_width}" mass="${wheel_mass}" distance_between_wheels="${base_length}"

File: carmen_description/urdf/sensors/camera.urdf.xacro (robot description, xacro)
@@ -1,7 +1,6 @@
 <robot xmlns:xacro="http://ros.org/wiki/xacro">
-    <xacro:property name="camera_radius" value="0.025"/>
     <xacro:property name="camera_size" value="0.03"/>
-    <xacro:property name="camera_mass"   value="0.1"/>
-    <xacro:macro name="simple_camera" params="prefix parent_link_name parent_length parent_height side">
+    <xacro:property name="camera_mass" value="0.1"/>
+    <xacro:macro name="simple_camera" params="prefix parent_link_name parent_length parent_height side x">
         <link name="${prefix}_camera_link">
             <visual>
@@ -13,5 +12,5 @@
         </link>
         <joint name="${prefix}_camera_joint" type="fixed">
-            <origin xyz="0 ${side * parent_length / 2} ${(parent_height + camera_size) / 2}"
+            <origin xyz="${x - camera_size / 2} ${side * parent_length / 2} ${(parent_height + camera_size) / 2}"
                     rpy="0 0 0"/>
             <parent link="${parent_link_name}"/>

File: carmen_description/urdf/sensors/sonar.urdf.xacro (robot description, xacro)
@@ -2,9 +2,9 @@
     <xacro:property name="sonar_size" value="0.03"/>
     <xacro:property name="sonar_mass" value="0.1"/>
-    <xacro:macro name="simple_sonar" params="prefix parent_link_name parent_length parent_height side">
+    <xacro:macro name="simple_sonar" params="prefix parent_link_name x y z x_side:=1 y_side:=1">
         <link name="${prefix}_sonar_link">
             <visual>
               <xacro:cube_geometry size="${sonar_size}"/>
-              <xacro:blue_material/>
+              <xacro:white_material/>
             </visual>
             <xacro:cube_collision size="${sonar_size}"/>
@@ -12,5 +12,5 @@
         </link>
         <joint name="${prefix}_sonar_joint" type="fixed">
-            <origin xyz="0 ${side * parent_length / 2} ${(parent_height + sonar_size) / 2}"
+            <origin xyz="${x - x_side * sonar_size / 2} ${y - y_side * sonar_size / 2} ${z + sonar_size / 2}"
                     rpy="0 0 0"/>
             <parent link="${parent_link_name}"/>

Commit message: Refactored base_link and base_footprint relation. Added sensor fusion of controller with IMU.

File: carmen_description/robot/carmen.gazebo.xacro (robot description, xacro)
@@ -210,5 +210,5 @@
             <robotNamespace>/</robotNamespace>
             <updateRate>50.0</updateRate>
-            <bodyName>base_footprint</bodyName>
+            <bodyName>base_link</bodyName>
             <frameId>imu_link</frameId>
             <topicName>imu/data</topicName>

File: carmen_description/robot/robot.urdf.xacro (robot description, xacro)
@@ -15,10 +15,4 @@
   <xacro:property name="imu_mass" value="0.01"/>
   <xacro:property name="bearing_radius" value="0.005"/>
-  <link name="base_footprint"/>
-  <joint name="base_footprint_joint" type="fixed">
-    <origin rpy="0 0 0" xyz="0 0 ${base_height / 2 + wheel_radius - bearing_radius}"/>
-    <parent link="base_footprint"/>
-    <child link="base_link"/>
-  </joint>
   <link name="base_link">
     <visual>
@@ -27,6 +21,19 @@
     </visual>
     <xacro:box_collision width="${base_width}" length="${base_length}" height="${base_height}"/>
+  </link>
+  <link name="base_footprint"/>
+  <joint name="base_footprint_joint" type="fixed">
+    <origin rpy="0 0 0" xyz="0 0 ${- base_height / 2 - wheel_radius + bearing_radius}"/>
+    <parent link="base_link"/>
+    <child link="base_footprint"/>
+  </joint>
+  <link name="inertial_link">
     <xacro:box_inertia width="${base_width}" length="${base_length}" height="${base_height}" mass="${base_mass}"/>
   </link>
+  <joint name="inertial_joint" type="fixed">
+    <origin xyz="0 0 0" rpy="0 0 0" />
+    <parent link="base_link" />
+    <child link="inertial_link" />
+  </joint>
   <link name="imu_link">
     <visual>
