Commit message: Added sensors (#3)
* Fixed differential drive controller.

* Added cameras and sonar xacro

* Added visualization of sonar, camera and IMU.

* Added simulation of all sensors

* Refactored base_link and base_footprint relation.
Added sensor fusion of controller with IMU.

* Fixed new line.

File: carmen_description/robot/carmen.gazebo.xacro (robot description, xacro)
@@ -12,61 +12,212 @@
     </gazebo>
     <gazebo reference="base_link">
+        <material>Gazebo/Yellow</material>
+    </gazebo>
+    <gazebo reference="front_left_wheel">
+        <mu1 value="1.0"/>
+        <mu2 value="1.0"/>
+        <kp value="10000000.0"/>
+        <kd value="1.0"/>
+        <fdir1 value="1 0 0"/>
+        <material>Gazebo/Black</material>
+    </gazebo>
+    <gazebo reference="front_right_wheel">
+        <mu1 value="1.0"/>
+        <mu2 value="1.0"/>
+        <kp value="10000000.0"/>
+        <kd value="1.0"/>
+        <fdir1 value="1 0 0"/>
+        <material>Gazebo/Black</material>
+    </gazebo>
+    <gazebo reference="rear_left_wheel">
+        <mu1 value="1.0"/>
+        <mu2 value="1.0"/>
+        <kp value="10000000.0"/>
+        <kd value="1.0"/>
+        <fdir1 value="1 0 0"/>
+        <material>Gazebo/Black</material>
+    </gazebo>
+    <gazebo reference="rear_right_wheel">
+        <mu1 value="1.0"/>
+        <mu2 value="1.0"/>
+        <kp value="10000000.0"/>
+        <kd value="1.0"/>
+        <fdir1 value="1 0 0"/>
+        <material>Gazebo/Black</material>
+    </gazebo>
+    <gazebo reference="front_right_bearing">
+        <mu1 value="1.0"/>
+        <mu2 value="1.0"/>
+        <kp value="10000000.0"/>
+        <kd value="1.0"/>
+        <material>Gazebo/Blue</material>
+    </gazebo>
+    <gazebo reference="front_left_bearing">
+        <mu1 value="1.0"/>
+        <mu2 value="1.0"/>
+        <kp value="10000000.0"/>
+        <kd value="1.0"/>
+        <material>Gazebo/Blue</material>
+    </gazebo>
+    <gazebo reference="rear_left_bearing">
+        <mu1 value="1.0"/>
+        <mu2 value="1.0"/>
+        <kp value="10000000.0"/>
+        <kd value="1.0"/>
+        <material>Gazebo/Blue</material>
+    </gazebo>
+    <gazebo reference="rear_right_bearing">
+        <mu1 value="1.0"/>
+        <mu2 value="1.0"/>
+        <kp value="10000000.0"/>
+        <kd value="1.0"/>
+        <material>Gazebo/Blue</material>
+    </gazebo>
+    <gazebo reference="left_sonar_link">
         <material>Gazebo/White</material>
-    </gazebo>
-    <gazebo reference="front_left_wheel">
-        <mu1 value="1.0"/>
-        <mu2 value="1.0"/>
-        <kp value="10000000.0"/>
-        <kd value="1.0"/>
-        <material>Gazebo/Black</material>
-    </gazebo>
-    <gazebo reference="front_right_wheel">
-        <mu1 value="1.0"/>
-        <mu2 value="1.0"/>
-        <kp value="10000000.0"/>
-        <kd value="1.0"/>
-        <material>Gazebo/Black</material>
-    </gazebo>
-    <gazebo reference="rear_left_wheel">
-        <mu1 value="1.0"/>
-        <mu2 value="1.0"/>
-        <kp value="10000000.0"/>
-        <kd value="1.0"/>
-        <material>Gazebo/Black</material>
-    </gazebo>
-    <gazebo reference="rear_right_wheel">
-        <mu1 value="1.0"/>
-        <mu2 value="1.0"/>
-        <kp value="10000000.0"/>
-        <kd value="1.0"/>
-        <material>Gazebo/Black</material>
-    </gazebo>
-    <gazebo reference="front_right_bearing">
-        <mu1 value="1.0"/>
-        <mu2 value="1.0"/>
-        <kp value="10000000.0"/>
-        <kd value="1.0"/>
-        <material>Gazebo/Blue</material>
-    </gazebo>
-    <gazebo reference="front_left_bearing">
-        <mu1 value="1.0"/>
-        <mu2 value="1.0"/>
-        <kp value="10000000.0"/>
-        <kd value="1.0"/>
-        <material>Gazebo/Blue</material>
-    </gazebo>
-    <gazebo reference="rear_left_bearing">
-        <mu1 value="1.0"/>
-        <mu2 value="1.0"/>
-        <kp value="10000000.0"/>
-        <kd value="1.0"/>
-        <material>Gazebo/Blue</material>
-    </gazebo>
-    <gazebo reference="rear_right_bearing">
-        <mu1 value="1.0"/>
-        <mu2 value="1.0"/>
-        <kp value="10000000.0"/>
-        <kd value="1.0"/>
-        <material>Gazebo/Blue</material>
+        <sensor type="ray" name="left_sonar">
+            <always_on>true</always_on>
+            <update_rate>40</update_rate>
+            <pose>0 0 0 0 0 0</pose>
+            <visualize>false</visualize>
+            <ray>
+                <scan>
+                    <horizontal>
+                        <samples>1</samples>
+                        <resolution>1</resolution>
+                        <min_angle>-0.13</min_angle>
+                        <max_angle>0.13</max_angle>
+                    </horizontal>
+                    <vertical>
+                        <samples>1</samples>
+                        <resolution>1</resolution>
+                        <min_angle>-0.13</min_angle>
+                        <max_angle>0.13</max_angle>
+                    </vertical>
+                </scan>
+                <range>
+                    <min>0.02</min>
+                    <max>4</max>
+                    <resolution>0.003</resolution>
+                </range>
+            </ray>
+            <plugin name="gazebo_ros_left_sonar_controller" filename="libhector_gazebo_ros_sonar.so">
+                <gaussianNoise>0.005</gaussianNoise>
+                <topicName>left_sonar</topicName>
+                <frameId>left_sonar_link</frameId>
+            </plugin>
+        </sensor>
+    </gazebo>
+    <gazebo reference="right_sonar_link">
+        <material>Gazebo/White</material>
+        <sensor type="ray" name="right_sonar">
+            <always_on>true</always_on>
+            <update_rate>40</update_rate>
+            <pose>0 0 0 0 0 0</pose>
+            <visualize>false</visualize>
+            <ray>
+                <scan>
+                    <horizontal>
+                        <samples>1</samples>
+                        <resolution>1</resolution>
+                        <min_angle>-0.13</min_angle>
+                        <max_angle>0.13</max_angle>
+                    </horizontal>
+                    <vertical>
+                        <samples>1</samples>
+                        <resolution>1</resolution>
+                        <min_angle>-0.13</min_angle>
+                        <max_angle>0.13</max_angle>
+                    </vertical>
+                </scan>
+                <range>
+                    <min>0.02</min>
+                    <max>4</max>
+                    <resolution>0.003</resolution>
+                </range>
+            </ray>
+            <plugin name="gazebo_ros_right_sonar_controller" filename="libhector_gazebo_ros_sonar.so">
+                <gaussianNoise>0.005</gaussianNoise>
+                <topicName>right_sonar</topicName>
+                <frameId>right_sonar_link</frameId>
+            </plugin>
+        </sensor>
+    </gazebo>
+    <gazebo reference="left_camera_link">
+        <material>Gazebo/Green</material>
+        <sensor type="multicamera" name="stereo_camera">
+            <update_rate>30.0</update_rate>
+            <camera name="left">
+                <horizontal_fov>1.3962634</horizontal_fov>
+                <image>
+                    <width>800</width>
+                    <height>800</height>
+                    <format>R8G8B8</format>
+                </image>
+                <clip>
+                    <near>0.02</near>
+                    <far>300</far>
+                </clip>
+                <noise>
+                    <type>gaussian</type>
+                    <mean>0.0</mean>
+                    <stddev>0.007</stddev>
+                </noise>
+            </camera>
+            <camera name="right">
+                <pose>0 -0.07 0 0 0 0</pose>
+                <horizontal_fov>1.3962634</horizontal_fov>
+                <image>
+                    <width>800</width>
+                    <height>800</height>
+                    <format>R8G8B8</format>
+                </image>
+                <clip>
+                    <near>0.02</near>
+                    <far>300</far>
+                </clip>
+                <noise>
+                    <type>gaussian</type>
+                    <mean>0.0</mean>
+                    <stddev>0.007</stddev>
+                </noise>
+            </camera>
+            <plugin name="stereo_camera_controller" filename="libgazebo_ros_multicamera.so">
+                <alwaysOn>true</alwaysOn>
+                <updateRate>0.0</updateRate>
+                <cameraName>stereocamera</cameraName>
+                <imageTopicName>image_raw</imageTopicName>
+                <cameraInfoTopicName>camera_info</cameraInfoTopicName>
+                <frameName>left_camera_link</frameName>
+                <rightFrameName>right_camera_link</rightFrameName>
+                <hackBaseline>0.07</hackBaseline>
+                <distortionK1>0.0</distortionK1>
+                <distortionK2>0.0</distortionK2>
+                <distortionK3>0.0</distortionK3>
+                <distortionT1>0.0</distortionT1>
+                <distortionT2>0.0</distortionT2>
+            </plugin>
+        </sensor>
+    </gazebo>
+    <gazebo reference="right_camera_link">
+        <material>Gazebo/Green</material>
+    </gazebo>
+    <gazebo reference="imu_link">
+        <material>Gazebo/Black</material>
+    </gazebo>
+    <gazebo>
+        <plugin name="imu_controller" filename="libhector_gazebo_ros_imu.so">
+            <robotNamespace>/</robotNamespace>
+            <updateRate>50.0</updateRate>
+            <bodyName>base_link</bodyName>
+            <frameId>imu_link</frameId>
+            <topicName>imu/data</topicName>
+            <accelDrift>0.005 0.005 0.005</accelDrift>
+            <accelGaussianNoise>0.005 0.005 0.005</accelGaussianNoise>
+            <rateDrift>0.00005 0.00005 0.00005</rateDrift>
+            <rateGaussianNoise>0.00005 0.00005 0.00005</rateGaussianNoise>
+            <headingDrift>0.005</headingDrift>
+            <headingGaussianNoise>0.005</headingGaussianNoise>
+        </plugin>
     </gazebo>
 </robot>

File: carmen_description/robot/robot.urdf.xacro (robot description, xacro)
@@ -3,4 +3,5 @@
   <xacro:include filename="$(find carmen_description)/urdf/common.urdf.xacro"/>
   <xacro:include filename="$(find carmen_description)/urdf/sensors/camera.urdf.xacro"/>
+  <xacro:include filename="$(find carmen_description)/urdf/sensors/sonar.urdf.xacro"/>
   <xacro:include filename="$(find carmen_description)/urdf/wheels.urdf.xacro"/>
   <xacro:property name="base_width" value="0.3"/>
@@ -11,19 +12,49 @@
   <xacro:property name="wheel_radius" value="0.035"/>
   <xacro:property name="wheel_mass" value="1"/>
+  <xacro:property name="imu_size" value="0.01"/>
+  <xacro:property name="imu_mass" value="0.01"/>
   <xacro:property name="bearing_radius" value="0.005"/>
-  <link name="base_footprint"/>
-  <joint name="base_footprint_joint" type="fixed">
-    <origin rpy="0 0 0" xyz="0 0 ${base_height / 2 + wheel_radius - bearing_radius}"/>
-    <parent link="base_footprint"/>
-    <child link="base_link"/>
-  </joint>
   <link name="base_link">
     <visual>
       <xacro:box_geometry width="${base_width}" length="${base_length}" height="${base_height}"/>
-      <xacro:navajo_white_material/>
+      <xacro:yellow_material/>
     </visual>
     <xacro:box_collision width="${base_width}" length="${base_length}" height="${base_height}"/>
+  </link>
+  <link name="base_footprint"/>
+  <joint name="base_footprint_joint" type="fixed">
+    <origin rpy="0 0 0" xyz="0 0 ${- base_height / 2 - wheel_radius + bearing_radius}"/>
+    <parent link="base_link"/>
+    <child link="base_footprint"/>
+  </joint>
+  <link name="inertial_link">
     <xacro:box_inertia width="${base_width}" length="${base_length}" height="${base_height}" mass="${base_mass}"/>
   </link>
+  <joint name="inertial_joint" type="fixed">
+    <origin xyz="0 0 0" rpy="0 0 0" />
+    <parent link="base_link" />
+    <child link="inertial_link" />
+  </joint>
+  <link name="imu_link">
+    <visual>
+      <xacro:cube_geometry size="${imu_size}"/>
+      <xacro:black_material/>
+    </visual>
+    <xacro:cube_collision size="${imu_size}"/>
+    <xacro:cube_inertia mass="${imu_mass}" size="${imu_size}"/>
+  </link>
+  <joint name="imu_joint" type="fixed">
+      <origin xyz="-0.025 0 ${(base_height + imu_size) / 2}" rpy="0 0 0"/>
+      <parent link="base_link"/>
+      <child link="imu_link"/>
+  </joint>
+  <xacro:simple_camera prefix="left" parent_link_name="base_link" parent_height="${base_height}"
+                       parent_length="${base_length / 2}" side="1" x="${base_width / 2}"/>
+  <xacro:simple_camera prefix="right" parent_link_name="base_link" parent_height="${base_height}"
+                       parent_length="${base_length / 2}" side="-1" x="${base_width / 2}"/>
+  <xacro:simple_sonar prefix="left" parent_link_name="base_link" x="${base_width / 2}" y="${base_length / 2}"
+                      z="${base_height / 2}"/>
+  <xacro:simple_sonar prefix="right" parent_link_name="base_link" x="${base_width / 2}" y="${-base_length / 2}"
+                      y_side="-1" z="${base_height / 2}"/>
   <xacro:wheel prefix="front_left" direction="1" bearing_radius="${bearing_radius}" radius="${wheel_radius}"
                width="${wheel_width}" mass="${wheel_mass}" distance_between_wheels="${base_length}"

Commit message: Added extra ultrasonic sensor to simulation and URDF. Added RangeSensorController to represent three ultrasonic sensors.

File: carmen_description/robot/carmen.gazebo.xacro (robot description, xacro)
@@ -106,4 +106,39 @@
                 <topicName>left_sonar</topicName>
                 <frameId>left_sonar_link</frameId>
+            </plugin>
+        </sensor>
+    </gazebo>
+    <gazebo reference="central_sonar_link">
+        <material>Gazebo/White</material>
+        <sensor type="ray" name="left_sonar">
+            <always_on>true</always_on>
+            <update_rate>40</update_rate>
+            <pose>0 0 0 0 0 0</pose>
+            <visualize>false</visualize>
+            <ray>
+                <scan>
+                    <horizontal>
+                        <samples>1</samples>
+                        <resolution>1</resolution>
+                        <min_angle>-0.13</min_angle>
+                        <max_angle>0.13</max_angle>
+                    </horizontal>
+                    <vertical>
+                        <samples>1</samples>
+                        <resolution>1</resolution>
+                        <min_angle>-0.13</min_angle>
+                        <max_angle>0.13</max_angle>
+                    </vertical>
+                </scan>
+                <range>
+                    <min>0.02</min>
+                    <max>4</max>
+                    <resolution>0.003</resolution>
+                </range>
+            </ray>
+            <plugin name="gazebo_ros_central_sonar_controller" filename="libhector_gazebo_ros_sonar.so">
+                <gaussianNoise>0.005</gaussianNoise>
+                <topicName>central_sonar</topicName>
+                <frameId>central_sonar_link</frameId>
             </plugin>
         </sensor>

File: carmen_description/robot/robot.urdf.xacro (robot description, xacro)
@@ -55,4 +55,6 @@
   <xacro:simple_sonar prefix="left" parent_link_name="base_link" x="${base_width / 2}" y="${base_length / 2}"
                       z="${base_height / 2}"/>
+  <xacro:simple_sonar prefix="central" parent_link_name="base_link" x="${base_width / 2}" y="0"
+                      z="${base_height / 2}"/>
   <xacro:simple_sonar prefix="right" parent_link_name="base_link" x="${base_width / 2}" y="${-base_length / 2}"
                       y_side="-1" z="${base_height / 2}"/>

Commit message: Added lidar to simulation. Added missing dependency.

File: carmen_description/robot/carmen.gazebo.xacro (robot description, xacro)
@@ -256,3 +256,35 @@
         </plugin>
     </gazebo>
+    <gazebo reference="lidar_link">
+      <material>Gazebo/Black</material>
+      <sensor type="gpu_ray" name="lidar_sensor">
+        <pose>0 0 0 0 0 0</pose>
+        <visualize>false</visualize>
+        <update_rate>40</update_rate>
+        <ray>
+          <scan>
+            <horizontal>
+              <samples>720</samples>
+              <resolution>1</resolution>
+              <min_angle>-1.570796</min_angle>
+              <max_angle>1.570796</max_angle>
+            </horizontal>
+          </scan>
+          <range>
+            <min>0.10</min>
+            <max>30.0</max>
+            <resolution>0.01</resolution>
+          </range>
+          <noise>
+            <type>gaussian</type>
+            <mean>0.0</mean>
+            <stddev>0.01</stddev>
+          </noise>
+        </ray>
+        <plugin name="gazebo_ros_lidar_controller" filename="libgazebo_ros_gpu_laser.so">
+          <topicName>/scan</topicName>
+          <frameName>lidar_link</frameName>
+        </plugin>
+      </sensor>
+    </gazebo>
 </robot>

Commit message: Added gmapping.

File: carmen_description/robot/carmen.gazebo.xacro (robot description, xacro)
@@ -283,5 +283,5 @@
         </ray>
         <plugin name="gazebo_ros_lidar_controller" filename="libgazebo_ros_gpu_laser.so">
-          <topicName>/scan</topicName>
+          <topicName>/laser/scan</topicName>
           <frameName>lidar_link</frameName>
         </plugin>

File: carmen_description/robot/robot.urdf.xacro (robot description, xacro)
@@ -14,5 +14,5 @@
   <xacro:property name="imu_size" value="0.01"/>
   <xacro:property name="imu_mass" value="0.01"/>
-  <xacro:property name="lidar_size" value="0.01"/>
+  <xacro:property name="lidar_size" value="0.05"/>
   <xacro:property name="lidar_mass" value="0.1"/>
   <xacro:property name="bearing_radius" value="0.005"/>
@@ -60,5 +60,5 @@
   </link>
   <joint name="lidar_joint" type="fixed">
-      <origin xyz="-0.025 0 ${(base_height + lidar_size) / 2}" rpy="0 0 0"/>
+      <origin xyz="-0.025 0 ${(base_height + lidar_size + lidar_size) / 2}" rpy="0 0 0"/>
       <parent link="base_link"/>
       <child link="lidar_link"/>
