Commit message: Added lidar to URDF

File: carmen_description/robot/robot.urdf.xacro (robot description, xacro)
@@ -14,4 +14,6 @@
   <xacro:property name="imu_size" value="0.01"/>
   <xacro:property name="imu_mass" value="0.01"/>
+  <xacro:property name="lidar_size" value="0.01"/>
+  <xacro:property name="lidar_mass" value="0.1"/>
   <xacro:property name="bearing_radius" value="0.005"/>
   <link name="base_link">
@@ -49,4 +51,17 @@
       <child link="imu_link"/>
   </joint>
+  <link name="lidar_link">
+    <visual>
+      <xacro:cube_geometry size="${lidar_size}"/>
+      <xacro:black_material/>
+    </visual>
+    <xacro:cube_collision size="${lidar_size}"/>
+    <xacro:cube_inertia mass="${lidar_mass}" size="${lidar_size}"/>
+  </link>
+  <joint name="lidar_joint" type="fixed">
+      <origin xyz="-0.025 0 ${(base_height + lidar_size) / 2}" rpy="0 0 0"/>
+      <parent link="base_link"/>
+      <child link="lidar_link"/>
+  </joint>
   <xacro:simple_camera prefix="left" parent_link_name="base_link" parent_height="${base_height}"
                        parent_length="${base_length / 2}" side="1" x="${base_width / 2}"/>

Commit message: Fixed lidar orientation.

File: carmen_description/robot/robot.urdf.xacro (robot description, xacro)
@@ -60,5 +60,5 @@
   </link>
   <joint name="lidar_joint" type="fixed">
-      <origin xyz="-0.025 0 ${(base_height + lidar_size + lidar_size) / 2}" rpy="0 0 0"/>
+      <origin xyz="-0.025 0 ${(base_height + lidar_size + lidar_size) / 2}" rpy="0 0 ${pi}"/>
       <parent link="base_link"/>
       <child link="lidar_link"/>

Commit message: Fixed IMU orientation and control depencencies.

File: carmen_description/robot/robot.urdf.xacro (robot description, xacro)
@@ -47,5 +47,5 @@
   </link>
   <joint name="imu_joint" type="fixed">
-      <origin xyz="-0.025 0 ${(base_height + imu_size) / 2}" rpy="0 0 0"/>
+      <origin xyz="-0.025 0 ${(base_height + imu_size) / 2}" rpy="0 0 ${pi / 2}"/>
       <parent link="base_link"/>
       <child link="imu_link"/>
